File: PCB and Case/snes_visualization_combi.brd (EAGLE design)
At the start: 116.8 x 33.5 mm, 22 parts, among them U1 TLC59282

Commit message: rerouted vis board, rev2 cleanups
Parts:
- moved JP4 51.0 mm to (113.0, 25.4)
- moved JP3 50.7 mm to (110.5, 27.9)
- moved C3 48.6 mm to (84.2, 19.8)
- moved R13 48.6 mm to (80.0, 19.8)
- moved U1 48.6 mm to (82.0, 25.3)
- moved LED3 45.3 mm to (73.9, 12.3)
- moved LED1 45.3 mm to (19.9, 29.9)
- moved LED10 45.3 mm to (19.9, 24.6)
- moved LED11 45.3 mm to (30.8, 16.8)
- moved LED12 45.3 mm to (19.9, 9.04)
- moved LED13 45.3 mm to (3.74, 16.8)
- moved LED14 45.3 mm to (19.9, 3.70)
- moved LED2 45.3 mm to (36.1, 16.8)
- moved LED4 45.3 mm to (58.3, 12.3)
- moved LED9 45.3 mm to (9.07, 16.8)
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Routing:
- net +3V3: track 226.1 -> 3.27 mm, vias 0 -> 1
- net ID2_LED: track 70.7 -> 92.6 mm
- net ID4_LED: track 68.7 -> 47.3 mm, vias 1 -> 0
- net DOWN_LED: track 39.1 -> 60.0 mm, vias 1 -> 0
- net LEFT_LED: track 51.8 -> 37.1 mm, vias 1 -> 0
- net ID1_LED: track 76.6 -> 88.3 mm
- net GND: track 22.9 -> 32.1 mm
- net ID3_LED: track 72.3 -> 65.2 mm, vias 1 -> 0
- net X_LED: track 60.5 -> 66.8 mm, vias 0 -> 1
- net UP_LED: track 20.9 -> 26.7 mm, vias 1 -> 0
- net R_LED: track 74.8 -> 80.4 mm, vias 1 -> 0
- net Y_LED: track 49.1 -> 54.6 mm, vias 0 -> 1
- net RIGHT_LED: track 20.6 -> 15.3 mm, vias 1 -> 0
- net L_LED: track 30.8 -> 35.6 mm
- net B_LED: track 86.8 -> 83.2 mm, vias 1 -> 0
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- added copper zone on layer 1, net +3V3
Other:
- board text added: "SNES Visualization"
- board text added: "TAStm32 remix rev1"
- board text removed: "SNES Visualization v1"
