File: PCB and Case/TAStm32_v4.sch (EAGLE design)
At the start: 55 parts, among them CN1 330pF, CN2 330pF, CN3 330pF, CN4 330pF, IC1 74HCT3G07DP-Q100H, IC2 74HCT3G07DP-Q100H, IC3 74AVCH4T245PW,118, IC4 74AVCH4T245PW,118, J1 ZX62D-B-5PA8, J10 RJSSE538002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

Commit message: more board tidyups
Parts:
- C15, C17: value 100nF -> 4.7uF
- S1, S2, S3, S4: value SWITCHN -> 3-1825910-1_SWITCHN; device 3-1825910-1:SWITCHN -> TAStm32_v4:3-1825910-1_SWITCHN
Connections:
- net GND: now also S1.P$2, S2.P$2; no longer S1.P$1, S2.P$1
- net SWITCH1: now also S1.P$1; no longer S1.P$2
- net SWITCH2: now also S2.P$1; no longer S2.P$2
Other:
- note removed: "Add insurance caps to outputs (maybe arrays)"
- note removed: "Add larger caps to console 5v rails, maybe"
- note removed: "Label debug pins"
- note removed: "Switch pads slightly wrong"
- note removed: "make D2 able to be read from schmitt-triggered inputs (NES/SNES) or voltage translators (N64)"
- note removed: "maybe omit pullups?"
Changed lines of the file:
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@@
 <part name="J11" library="TAStm32_v4" deviceset="RJSSE538002_RJSSE538002" device="" package3d_urn="urn:adsk.eagle:package:18856791/2" value="RJSSE538002"/>
 <part name="J4" library="TAStm32_v4" deviceset="SAMTEC-TSM-102-01-X-SH_SAMTEC-TSM-102-01-X-SH" device="" package3d_urn="urn:adsk.eagle:package:18856692/2" value="CONSOLE_RESET"/>
-<part name="S1" library="3-1825910-1" deviceset="SWITCHN" device="" override_package3d_urn="urn:adsk.eagle:package:25997948/2" override_package_urn="urn:adsk.eagle:footprint:25997949/1"/>
-<part name="S2" library="3-1825910-1" deviceset="SWITCHN" device="" override_package3d_urn="urn:adsk.eagle:package:25998021/2" override_package_urn="urn:adsk.eagle:footprint:25998023/1"/>
-<part name="S3" library="3-1825910-1" deviceset="SWITCHN" device="" override_package3d_urn="urn:adsk.eagle:package:25998025/2" override_package_urn="urn:adsk.eagle:footprint:25998026/1"/>
-<part name="S4" library="3-1825910-1" deviceset="SWITCHN" device="" override_package3d_urn="urn:adsk.eagle:package:25998028/2" override_package_urn="urn:adsk.eagle:footprint:25998029/1"/>
 <part name="J2" library="SamacSys_Parts" deviceset="UE27-AC54-100" device="" override_package3d_urn="urn:adsk.eagle:package:25997941/2" override_package_urn="urn:adsk.eagle:footprint:25997942/1"/>
 <part name="D1" library="TAStm32_v4" deviceset="DIODE_BAT60J" device="" value="BAT60J"/>
@@
 <part name="C14" library="rcl" library_urn="urn:adsk.eagle:library:334" deviceset="C-EU" device="C0603K" package3d_urn="urn:adsk.eagle:package:23680/2" value="100nF"/>
 <part name="GND30" library="supply1" library_urn="urn:adsk.eagle:library:371" deviceset="GND" device=""/>
-<part name="C15" library="rcl" library_urn="urn:adsk.eagle:library:334" deviceset="C-EU" device="C0603K" package3d_urn="urn:adsk.eagle:package:23680/2" value="100nF"/>
+<part name="C15" library="rcl" library_urn="urn:adsk.eagle:library:334" deviceset="C-EU" device="C0603K" package3d_urn="urn:adsk.eagle:package:23680/2" value="4.7uF"/>
 <part name="GND31" library="supply1" library_urn="urn:adsk.eagle:library:371" deviceset="GND" device=""/>
 <part name="SUPPLY14" library="supply2" library_urn="urn:adsk.eagle:library:372" deviceset="V+" device=""/>
@@
 <part name="C16" library="rcl" library_urn="urn:adsk.eagle:library:334" deviceset="C-EU" device="C0603K" package3d_urn="urn:adsk.eagle:package:23680/2" value="100nF"/>
 <part name="GND34" library="supply1" library_urn="urn:adsk.eagle:library:371" deviceset="GND" device=""/>
-<part name="C17" library="rcl" library_urn="urn:adsk.eagle:library:334" deviceset="C-EU" device="C0603K" package3d_urn="urn:adsk.eagle:package:23680/2" value="100nF"/>
+<part name="C17" library="rcl" library_urn="urn:adsk.eagle:library:334" deviceset="C-EU" device="C0603K" package3d_urn="urn:adsk.eagle:package:23680/2" value="4.7uF"/>
 <part name="GND35" library="supply1" library_urn="urn:adsk.eagle:library:371" deviceset="GND" device=""/>
 <part name="SUPPLY20" library="supply2" library_urn="urn:adsk.eagle:library:372" deviceset="V+" device=""/>
@@
 <part name="GND39" library="supply1" library_urn="urn:adsk.eagle:library:371" deviceset="GND" device=""/>
 <part name="FRAME1" library="frames" library_urn="urn:adsk.eagle:library:229" deviceset="A3L-LOC" device=""/>
+<part name="S2" library="TAStm32_v4" deviceset="3-1825910-1_SWITCHN" device=""/>
+<part name="S1" library="TAStm32_v4" deviceset="3-1825910-1_SWITCHN" device=""/>
+<part name="S4" library="TAStm32_v4" deviceset="3-1825910-1_SWITCHN" device=""/>
+<part name="S3" library="TAStm32_v4" deviceset="3-1825910-1_SWITCHN" device=""/>
 </parts>
 <sheets>
@@
 <text x="320.04" y="233.68" size="2.54" layer="97">Controller Outputs</text>
 <text x="314.96" y="149.86" size="2.54" layer="97">Expansion/Vis Ports</text>
-<text x="180.34" y="17.78" size="1.778" layer="91">Switch pads slightly wrong</text>
-<text x="180.34" y="15.24" size="1.778" layer="91">Add larger caps to console 5v rails, maybe</text>
-<text x="180.34" y="12.7" size="1.778" layer="91">Add insurance caps to outputs (maybe arrays)</text>
-<text x="180.34" y="10.16" size="1.778" layer="91">Label debug pins</text>
-<text x="180.34" y="7.62" size="1.778" layer="91">make D2 able to be read from schmitt-triggered inputs (NES/SNES) or voltage translators (N64)</text>
-<text x="180.34" y="5.08" size="1.778" layer="91">maybe omit pullups?</text>
 <text x="210.82" y="246.38" size="2.54" layer="97">Input Buffers</text>
 <text x="215.9" y="119.38" size="2.54" layer="97">Output Buffers</text>
@@
 <instance part="J4" gate="A" x="358.14" y="48.26" smashed="yes">
 <attribute name="NAME" x="359.41" y="52.07" size="1.778" layer="95"/>
-</instance>
-<instance part="S1" gate="G$1" x="124.46" y="96.52" smashed="yes" rot="MR0">
-<attribute name="NAME" x="130.81" y="97.79" size="1.778" layer="95" rot="MR0" align="center-left"/>
-</instance>
-<instance part="S2" gate="G$1" x="124.46" y="99.06" smashed="yes" rot="MR0">
-<attribute name="NAME" x="130.81" y="100.33" size="1.778" layer="95" rot="MR0" align="center-left"/>
-</instance>
-<instance part="S3" gate="G$1" x="124.46" y="86.36" smashed="yes">
-<attribute name="NAME" x="128.27" y="87.63" size="1.778" layer="95" align="center-left"/>
-</instance>
-<instance part="S4" gate="G$1" x="124.46" y="88.9" smashed="yes">
-<attribute name="NAME" x="128.27" y="90.17" size="1.778" layer="95" align="center-left"/>
 </instance>
 <instance part="J2" gate="G$1" x="101.6" y="228.6" smashed="yes">
@@
 <attribute name="SHEET" x="357.505" y="5.08" size="2.54" layer="94"/>
 </instance>
+<instance part="S2" gate="G$1" x="124.46" y="99.06" smashed="yes">
+<attribute name="NAME" x="115.57" y="106.68" size="1.778" layer="95" align="center-left"/>
+<attribute name="VALUE" x="115.57" y="104.14" size="1.778" layer="96" align="center-left"/>
+</instance>
+<instance part="S1" gate="G$1" x="124.46" y="96.52" smashed="yes">
+<attribute name="NAME" x="115.57" y="104.14" size="1.778" layer="95" align="center-left"/>
+<attribute name="VALUE" x="115.57" y="101.6" size="1.778" layer="96" align="center-left"/>
+</instance>
+<instance part="S4" gate="G$1" x="124.46" y="88.9" smashed="yes">
+<attribute name="NAME" x="115.57" y="96.52" size="1.778" layer="95" align="center-left"/>
+<attribute name="VALUE" x="115.57" y="93.98" size="1.778" layer="96" align="center-left"/>
+</instance>
+<instance part="S3" gate="G$1" x="124.46" y="86.36" smashed="yes">
+<attribute name="NAME" x="115.57" y="93.98" size="1.778" layer="95" align="center-left"/>
+<attribute name="VALUE" x="115.57" y="91.44" size="1.778" layer="96" align="center-left"/>
+</instance>
 </instances>
 <busses>
@@
 </segment>
 <segment>
+<wire x1="132.08" y1="88.9" x2="132.08" y2="86.36" width="0.1524" layer="91"/>
+<pinref part="GND2" gate="1" pin="GND"/>
 <pinref part="S4" gate="G$1" pin="P$2"/>
 <pinref part="S3" gate="G$1" pin="P$2"/>
-<wire x1="132.08" y1="88.9" x2="132.08" y2="86.36" width="0.1524" layer="91"/>
-<pinref part="GND2" gate="1" pin="GND"/>
 <junction x="132.08" y="86.36"/>
 </segment>
 <segment>
-<pinref part="S2" gate="G$1" pin="P$1"/>
-<pinref part="S1" gate="G$1" pin="P$1"/>
 <wire x1="132.08" y1="99.06" x2="132.08" y2="96.52" width="0.1524" layer="91"/>
 <pinref part="GND11" gate="1" pin="GND"/>
+<pinref part="S2" gate="G$1" pin="P$2"/>
+<pinref part="S1" gate="G$1" pin="P$2"/>
 <junction x="132.08" y="96.52"/>
 </segment>
@@
 <net name="SWITCH4" class="0">
 <segment>
-<pinref part="S4" gate="G$1" pin="P$1"/>
 <wire x1="116.84" y1="88.9" x2="114.3" y2="88.9" width="0.1524" layer="91"/>
 <label x="114.3" y="88.9" size="1.778" layer="95" rot="R180"/>
+<pinref part="S4" gate="G$1" pin="P$1"/>
 </segment>
 <segment>
@@
 <net name="SWITCH3" class="0">
 <segment>
-<pinref part="S3" gate="G$1" pin="P$1"/>
 <wire x1="116.84" y1="86.36" x2="114.3" y2="86.36" width="0.1524" layer="91"/>
 <label x="114.3" y="86.36" size="1.778" layer="95" rot="R180"/>
+<pinref part="S3" gate="G$1" pin="P$1"/>
 </segment>
 <segment>
@@
 <net name="SWITCH1" class="0">
 <segment>
-<pinref part="S1" gate="G$1" pin="P$2"/>
 <wire x1="116.84" y1="96.52" x2="114.3" y2="96.52" width="0.1524" layer="91"/>
 <label x="114.3" y="96.52" size="1.778" layer="95" rot="R180"/>
+<pinref part="S1" gate="G$1" pin="P$1"/>
 </segment>
 <segment>
@@
 <net name="SWITCH2" class="0">
 <segment>
-<pinref part="S2" gate="G$1" pin="P$2"/>
 <wire x1="116.84" y1="99.06" x2="114.3" y2="99.06" width="0.1524" layer="91"/>
 <label x="114.3" y="99.06" size="1.778" layer="95" rot="R180"/>
-</segment>
-<segment>
+<pinref part="S2" gate="G$1" pin="P$1"/>
+</segment>
+<segment>

Commit message: part number updates
Parts:
- IC1, IC2: value 74HCT3G07DP-Q100H -> 74LVC3G17DP
- IC3, IC4: value 74AVCH4T245PW,118 -> 74AXP4T245
- RN5: value 47K -> 47R
Other:
- moved on the sheet: RN5
Changed lines of the file:
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@@
 <part name="J3" library="TSM-105-02-L-SH" deviceset="TSM-105-02-L-SH" device="J"/>
 <part name="RN4" library="resistor-net" library_urn="urn:adsk.eagle:library:343" deviceset="CTS742C083" device="" package3d_urn="urn:adsk.eagle:package:24985/1" value="47R"/>
-<part name="RN5" library="resistor-net" library_urn="urn:adsk.eagle:library:343" deviceset="CTS742C083" device="" package3d_urn="urn:adsk.eagle:package:24985/1" value="47K"/>
+<part name="RN5" library="resistor-net" library_urn="urn:adsk.eagle:library:343" deviceset="CTS742C083" device="" package3d_urn="urn:adsk.eagle:package:24985/1" value="47R"/>
 <part name="C5" library="rcl" library_urn="urn:adsk.eagle:library:334" deviceset="C-EU" device="C0603K" package3d_urn="urn:adsk.eagle:package:23680/2" value="100nF"/>
 <part name="RN1" library="resistor-net" library_urn="urn:adsk.eagle:library:343" deviceset="CTS742C083" device="" package3d_urn="urn:adsk.eagle:package:24985/1" value="47K"/>
@@
 <part name="GND28" library="supply1" library_urn="urn:adsk.eagle:library:371" deviceset="GND" device=""/>
 <part name="RN3" library="resistor-net" library_urn="urn:adsk.eagle:library:343" deviceset="CTS742C083" device="" package3d_urn="urn:adsk.eagle:package:24985/1"/>
-<part name="IC1" library="SamacSys_Parts" deviceset="74HCT3G07DP-Q100H" device=""/>
-<part name="IC2" library="SamacSys_Parts" deviceset="74HCT3G07DP-Q100H" device=""/>
-<part name="IC3" library="SamacSys_Parts" deviceset="74AVCH4T245PW,118" device=""/>
+<part name="IC1" library="SamacSys_Parts" deviceset="74HCT3G07DP-Q100H" device="" value="74LVC3G17DP"/>
+<part name="IC2" library="SamacSys_Parts" deviceset="74HCT3G07DP-Q100H" device="" value="74LVC3G17DP"/>
+<part name="IC3" library="SamacSys_Parts" deviceset="74AVCH4T245PW,118" device="" value="74AXP4T245"/>
 <part name="SUPPLY13" library="supply2" library_urn="urn:adsk.eagle:library:372" deviceset="V+" device=""/>
 <part name="GND26" library="supply1" library_urn="urn:adsk.eagle:library:371" deviceset="GND" device=""/>
@@
 <part name="GND33" library="supply1" library_urn="urn:adsk.eagle:library:371" deviceset="GND" device=""/>
 <part name="RN7" library="resistor-net" library_urn="urn:adsk.eagle:library:343" deviceset="CTS742C083" device="" package3d_urn="urn:adsk.eagle:package:24985/1" value="47R"/>
-<part name="IC4" library="SamacSys_Parts" deviceset="74AVCH4T245PW,118" device=""/>
+<part name="IC4" library="SamacSys_Parts" deviceset="74AVCH4T245PW,118" device="" value="74AXP4T245"/>
 <part name="C16" library="rcl" library_urn="urn:adsk.eagle:library:334" deviceset="C-EU" device="C0603K" package3d_urn="urn:adsk.eagle:package:23680/2" value="100nF"/>
 <part name="GND34" library="supply1" library_urn="urn:adsk.eagle:library:371" deviceset="GND" device=""/>
@@
 <attribute name="VALUE" x="248.92" y="211.582" size="1.778" layer="96" rot="MR0"/>
 </instance>
-<instance part="RN5" gate="G$1" x="248.92" y="165.1" smashed="yes" rot="MR0">
-<attribute name="NAME" x="250.825" y="170.18" size="1.778" layer="95" rot="MR0"/>
-<attribute name="VALUE" x="251.46" y="155.702" size="1.778" layer="96" rot="MR0"/>
+<instance part="RN5" gate="G$1" x="243.84" y="160.02" smashed="yes" rot="R180">
+<attribute name="NAME" x="245.745" y="154.94" size="1.778" layer="95" rot="R180"/>
+<attribute name="VALUE" x="246.38" y="169.418" size="1.778" layer="96" rot="R180"/>
 </instance>
 <instance part="C5" gate="G$1" x="200.66" y="228.6" smashed="yes" rot="MR270">
@@
 <instance part="IC2" gate="G$1" x="215.9" y="167.64" smashed="yes" rot="MR0">
 <attribute name="NAME" x="215.9" y="170.18" size="1.778" layer="95" rot="MR0" align="center-left"/>
-<attribute name="VALUE" x="212.09" y="154.94" size="1.778" layer="96" rot="MR0" align="center-left"/>
+<attribute name="VALUE" x="212.09" y="152.4" size="1.778" layer="96" rot="MR0" align="center-left"/>
 </instance>
 <instance part="IC3" gate="G$1" x="185.42" y="109.22" smashed="yes">
@@
 </segment>
 <segment>
-<wire x1="254" y1="160.02" x2="256.54" y2="160.02" width="0.1524" layer="91"/>
-<label x="256.54" y="160.02" size="1.27" layer="95" rot="MR180" xref="yes"/>
+<wire x1="248.92" y1="165.1" x2="251.46" y2="165.1" width="0.1524" layer="91"/>
+<label x="251.46" y="165.1" size="1.27" layer="95" xref="yes"/>
 <pinref part="RN5" gate="G$1" pin="4"/>
 </segment>
@@
 </segment>
 <segment>
-<wire x1="254" y1="162.56" x2="256.54" y2="162.56" width="0.1524" layer="91"/>
-<label x="256.54" y="162.56" size="1.27" layer="95" rot="MR180" xref="yes"/>
+<wire x1="248.92" y1="162.56" x2="251.46" y2="162.56" width="0.1524" layer="91"/>
+<label x="251.46" y="162.56" size="1.27" layer="95" xref="yes"/>
 <pinref part="RN5" gate="G$1" pin="3"/>
 </segment>
@@
 </segment>
 <segment>
-<wire x1="254" y1="167.64" x2="256.54" y2="167.64" width="0.1524" layer="91"/>
-<label x="256.54" y="167.64" size="1.27" layer="95" xref="yes"/>
+<wire x1="248.92" y1="157.48" x2="251.46" y2="157.48" width="0.1524" layer="91"/>
+<label x="251.46" y="157.48" size="1.27" layer="95" rot="MR180" xref="yes"/>
 <pinref part="RN5" gate="G$1" pin="1"/>
 </segment>
@@
 </segment>
 <segment>
-<label x="187.96" y="213.36" size="1.27" layer="95" rot="MR0" xref="yes"/>
+<label x="187.96" y="210.82" size="1.27" layer="95" rot="MR0" xref="yes"/>
 <pinref part="IC1" gate="G$1" pin="3Y"/>
 <wire x1="215.9" y1="220.98" x2="203.2" y2="220.98" width="0.1524" layer="91"/>
-<wire x1="203.2" y1="220.98" x2="203.2" y2="213.36" width="0.1524" layer="91"/>
-<wire x1="187.96" y1="213.36" x2="203.2" y2="213.36" width="0.1524" layer="91"/>
+<wire x1="203.2" y1="220.98" x2="203.2" y2="210.82" width="0.1524" layer="91"/>
+<wire x1="187.96" y1="210.82" x2="203.2" y2="210.82" width="0.1524" layer="91"/>
 </segment>
 </net>
@@
 </segment>
 <segment>
-<label x="187.96" y="157.48" size="1.27" layer="95" rot="MR0" xref="yes"/>
+<label x="187.96" y="154.94" size="1.27" layer="95" rot="MR0" xref="yes"/>
 <pinref part="IC2" gate="G$1" pin="3Y"/>
-<wire x1="215.9" y1="165.1" x2="208.28" y2="165.1" width="0.1524" layer="91"/>
-<wire x1="208.28" y1="165.1" x2="208.28" y2="157.48" width="0.1524" layer="91"/>
-<wire x1="208.28" y1="157.48" x2="187.96" y2="157.48" width="0.1524" layer="91"/>
+<wire x1="215.9" y1="165.1" x2="203.2" y2="165.1" width="0.1524" layer="91"/>
+<wire x1="203.2" y1="165.1" x2="203.2" y2="154.94" width="0.1524" layer="91"/>
+<wire x1="203.2" y1="154.94" x2="187.96" y2="154.94" width="0.1524" layer="91"/>
 </segment>
 </net>
@@
 <wire x1="228.6" y1="220.98" x2="223.52" y2="220.98" width="0.1524" layer="91"/>
 <wire x1="223.52" y1="220.98" x2="220.98" y2="220.98" width="0.1524" layer="91"/>
-<wire x1="220.98" y1="220.98" x2="220.98" y2="210.82" width="0.1524" layer="91"/>
-<wire x1="220.98" y1="210.82" x2="172.72" y2="210.82" width="0.1524" layer="91"/>
-<wire x1="172.72" y1="210.82" x2="172.72" y2="218.44" width="0.1524" layer="91"/>
+<wire x1="220.98" y1="220.98" x2="220.98" y2="205.74" width="0.1524" layer="91"/>
+<wire x1="220.98" y1="205.74" x2="172.72" y2="205.74" width="0.1524" layer="91"/>
+<wire x1="172.72" y1="205.74" x2="172.72" y2="218.44" width="0.1524" layer="91"/>
 <pinref part="IC1" gate="G$1" pin="3A"/>
 <wire x1="172.72" y1="218.44" x2="190.5" y2="218.44" width="0.1524" layer="91"/>
@@
 <junction x="226.06" y="167.64"/>
 <pinref part="RN5" gate="G$1" pin="6"/>
-<wire x1="241.3" y1="162.56" x2="233.68" y2="162.56" width="0.1524" layer="91"/>
+<wire x1="236.22" y1="162.56" x2="233.68" y2="162.56" width="0.1524" layer="91"/>
 <wire x1="233.68" y1="162.56" x2="233.68" y2="167.64" width="0.1524" layer="91"/>
 <wire x1="233.68" y1="167.64" x2="228.6" y2="167.64" width="0.1524" layer="91"/>
@@
 <segment>
 <wire x1="220.98" y1="165.1" x2="231.14" y2="165.1" width="0.1524" layer="91"/>
-<wire x1="220.98" y1="165.1" x2="220.98" y2="157.48" width="0.1524" layer="91"/>
-<wire x1="220.98" y1="157.48" x2="220.98" y2="154.94" width="0.1524" layer="91"/>
-<wire x1="220.98" y1="154.94" x2="198.12" y2="154.94" width="0.1524" layer="91"/>
-<wire x1="198.12" y1="154.94" x2="198.12" y2="162.56" width="0.1524" layer="91"/>
+<wire x1="220.98" y1="157.48" x2="220.98" y2="149.86" width="0.1524" layer="91"/>
+<wire x1="220.98" y1="149.86" x2="172.72" y2="149.86" width="0.1524" layer="91"/>
+<wire x1="172.72" y1="149.86" x2="172.72" y2="162.56" width="0.1524" layer="91"/>
 <pinref part="IC2" gate="G$1" pin="3A"/>
-<wire x1="198.12" y1="162.56" x2="190.5" y2="162.56" width="0.1524" layer="91"/>
+<wire x1="172.72" y1="162.56" x2="190.5" y2="162.56" width="0.1524" layer="91"/>
 <pinref part="RN2" gate="G$1" pin="1"/>
 <wire x1="231.14" y1="170.18" x2="231.14" y2="165.1" width="0.1524" layer="91"/>
@@
 <wire x1="220.98" y1="157.48" x2="220.98" y2="165.1" width="0.1524" layer="91"/>
 <junction x="220.98" y="165.1"/>
-<wire x1="231.14" y1="165.1" x2="238.76" y2="165.1" width="0.1524" layer="91"/>
+<wire x1="231.14" y1="165.1" x2="236.22" y2="165.1" width="0.1524" layer="91"/>
 <junction x="231.14" y="165.1"/>
-<wire x1="238.76" y1="165.1" x2="238.76" y2="160.02" width="0.1524" layer="91"/>
 <pinref part="RN5" gate="G$1" pin="5"/>
-<wire x1="238.76" y1="160.02" x2="241.3" y2="160.02" width="0.1524" layer="91"/>
 <junction x="220.98" y="157.48"/>
 </segment>
@@
 <wire x1="231.14" y1="157.48" x2="231.14" y2="162.56" width="0.1524" layer="91"/>
 <pinref part="RN5" gate="G$1" pin="8"/>
-<wire x1="241.3" y1="167.64" x2="236.22" y2="167.64" width="0.1524" layer="91"/>
-<wire x1="236.22" y1="167.64" x2="236.22" y2="157.48" width="0.1524" layer="91"/>
 <wire x1="236.22" y1="157.48" x2="231.14" y2="157.48" width="0.1524" layer="91"/>
 <junction x="231.14" y="157.48"/>
